File: voltameter/voltameter.kicad_sch (KiCad schematic)
At the start: 0 parts

Commit message: refresh
Parts:
- added C1: 4.7u, Capacitor_THT:CP_Radial_D5.0mm_P2.50mm, symbol Device:C_Polarized
- added D1, D10, D2, D3, D4, D5, D6, D7, D8, D9: LED, LED_THT:LED_D5.0mm, symbol Device:LED
- added J1: Screw_Terminal_01x02, Connector_JST:JST_EH_S2B-EH_1x02_P2.50mm_Horizontal, symbol Connector:Screw_Terminal_01x02
- added R1: 1k, Resistor_THT:R_Axial_DIN0204_L3.6mm_D1.6mm_P1.90mm_Vertical, symbol Device:R_US
- added RV2: R_Potentiometer_US, Potentiometer_THT:Potentiometer_Alps_RK163_Single_Horizontal, symbol Device:R_Potentiometer_US
- added U1: 4017, Package_DIP:DIP-16_W7.62mm, symbol 4xxx:4017
- added U2: NE555P, Package_DIP:DIP-8_W7.62mm, symbol Timer:NE555P
Connections:
- new net: D6.2 (A), U1.1 (Q5)
- new net: D5.2 (A), U1.10 (Q4)
- new net: D10.2 (A), U1.11 (Q9)
- new net: U1.14 (CLK), U2.3 (OUT)
- new net: D2.2 (A), U1.2 (Q1)
- new net: D1.2 (A), U1.3 (Q0)
- new net: D3.2 (A), U1.4 (Q2)
- new net: D7.2 (A), U1.5 (Q6)
- new net: D8.2 (A), U1.6 (Q7)
- new net: D4.2 (A), U1.7 (Q3)
- new net: D9.2 (A), U1.9 (Q8)
- new net: D1.1 (K), D10.1 (K), D2.1 (K), D3.1 (K), D4.1 (K), D5.1 (K), D6.1 (K), D7.1 (K), D8.1 (K), D9.1 (K), R1.1
- new net: C1.1, RV2.3, U2.2 (TRIG), U2.6 (THRES)
- new net: RV2.2, U2.7 (DISCH)
- new net +9V: J1.2 (Pin_2), RV2.1, U1.16 (VDD), U2.8 (VCC)
- new net GND: C1.2, J1.1 (Pin_1), R1.2, U1.13 (CKEN), U1.15 (Reset), U1.8 (VSS), U2.1 (GND)
- no-connect marks 0 -> 3
