File: ring counter/ring counter.kicad_pcb (KiCad board)
At the start: 4 copper layers, 95.1 x 80 mm, 16 parts, among them J1 Screw_Terminal_01x02, U1 4017, U2 NE555P

Commit message: refresh
Other:
- copper layers 4 -> 2
